File: hardware/eagle/RB02.sch (EAGLE design)
At the start: 19 parts, among them J1 CON_TERMINAL_BLOCK_02-5MM, J2 CON_TERMINAL_BLOCK_02-5MM, J3 CON_TERMINAL_BLOCK_02-5MM, J4 CON_TERMINAL_BLOCK_02-5MM, K1 JS-M1A-12V-5, K2 JS-M1A-12V-5, Q1 BC547, Q2 BC547

Commit message: BC337s instead of BC546s
Parts:
- Q1, Q2: value BC547 -> BC337; device transistor-small-signal:BC547 -> transistor:BC337
Other:
- moved on the sheet: D1, J1, J2, K1, LED1, PCB1, R1, R2, R4

Commit message: JS-M1 relay package
Parts:
- K1, K2: value JS-M1A-12V-5 -> JS-M1-12V-5; device relay:JS-M1A-12V-5 -> relay:JS-M1-12V-5; MF (none) -> FARNELL; MPN (none) -> JSM1-12V-5; OC_FARNELL (none) -> 910351; OC_NEWARK (none) -> 14J1764
Changed lines of the file:
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@@
 <part name="J2" library="dp_devices" deviceset="CON_TERMINAL_BLOCK_02" device="-5MM"/>
 <part name="Q1" library="transistor" deviceset="BC337" device=""/>
-<part name="K1" library="relay" deviceset="JS-M1A*" device="" technology="-12V-5"/>
+<part name="K1" library="relay" deviceset="JS-M1*" device="" technology="-12V-5">
+<attribute name="MF" value="FARNELL"/>
+<attribute name="MPN" value="JSM1-12V-5"/>
+<attribute name="OC_FARNELL" value="910351"/>
+<attribute name="OC_NEWARK" value="14J1764"/>
+</part>
 <part name="P+1" library="supply1" deviceset="VCC" device=""/>
 <part name="P+2" library="supply1" deviceset="VCC" device=""/>
@@
 <part name="J4" library="dp_devices" deviceset="CON_TERMINAL_BLOCK_02" device="-5MM"/>
 <part name="Q2" library="transistor" deviceset="BC337" device=""/>
-<part name="K2" library="relay" deviceset="JS-M1A*" device="" technology="-12V-5"/>
+<part name="K2" library="relay" deviceset="JS-M1*" device="" technology="-12V-5">
+<attribute name="MF" value="FARNELL"/>
+<attribute name="MPN" value="JSM1-12V-5"/>
+<attribute name="OC_FARNELL" value="910351"/>
+<attribute name="OC_NEWARK" value="14J1764"/>
+</part>
 <part name="P+4" library="supply1" deviceset="VCC" device=""/>
 <part name="P+5" library="supply1" deviceset="VCC" device=""/>
@@
 <attribute name="PART" x="125.73" y="83.82" size="1.778" layer="95"/>
 </instance>
-<instance part="K1" gate="2" x="134.62" y="93.98" smashed="yes"/>
+<instance part="K1" gate="2" x="134.62" y="91.44" smashed="yes"/>
 <instance part="P+1" gate="VCC" x="76.2" y="142.24"/>
 <instance part="P+2" gate="VCC" x="101.6" y="106.68"/>
@@
 <attribute name="PART" x="125.73" y="147.32" size="1.778" layer="95"/>
 </instance>
-<instance part="K2" gate="2" x="134.62" y="157.48" smashed="yes"/>
+<instance part="K2" gate="2" x="134.62" y="154.94" smashed="yes"/>
 <instance part="P+4" gate="VCC" x="101.6" y="170.18"/>
 <instance part="P+5" gate="VCC" x="114.3" y="167.64"/>
@@
 <label x="144.78" y="154.94" size="1.778" layer="95"/>
 <pinref part="K2" gate="2" pin="S"/>
-<wire x1="134.62" y1="162.56" x2="142.24" y2="162.56" width="0.1524" layer="91"/>
+<wire x1="129.54" y1="160.02" x2="129.54" y2="162.56" width="0.1524" layer="91"/>
+<wire x1="129.54" y1="162.56" x2="142.24" y2="162.56" width="0.1524" layer="91"/>
 <wire x1="142.24" y1="162.56" x2="142.24" y2="154.94" width="0.1524" layer="91"/>
 <pinref part="J4" gate="CON" pin="1"/>
@@
 <label x="144.78" y="91.44" size="1.778" layer="95"/>
 <pinref part="K1" gate="2" pin="S"/>
-<wire x1="134.62" y1="99.06" x2="142.24" y2="99.06" width="0.1524" layer="91"/>
+<wire x1="129.54" y1="96.52" x2="129.54" y2="99.06" width="0.1524" layer="91"/>
+<wire x1="129.54" y1="99.06" x2="142.24" y2="99.06" width="0.1524" layer="91"/>
 <wire x1="142.24" y1="99.06" x2="142.24" y2="91.44" width="0.1524" layer="91"/>
 <pinref part="J2" gate="CON" pin="1"/>
