File: hardware/RD01/RD01.sch (EAGLE design)
At the start: 19 parts, among them J1 CON_TERMINAL_BLOCK_02-5MM, J2 CON_TERMINAL_BLOCK_02-5MM, J3 CON_TERMINAL_BLOCK_02-5MM, J4 CON_TERMINAL_BLOCK_02-5MM, K1 JS-M1-12V-5, K2 JS-M1-12V-5, Q1 BC337, Q2 BC337

Commit message: RD01 Elecrow order
Parts:
- J2, J4: value CON_TERMINAL_BLOCK_02-5MM -> CON_TERMINAL_BLOCK_03-5MM; device dp_devices:CON_TERMINAL_BLOCK_02-5MM -> dp_devices:CON_TERMINAL_BLOCK_03-5MM
- LED1, LED2: device SparkFun:LED5MM -> dp_devices:LED-3MM
Connections:
- net LOAD_A2 renamed LOAD_A_C
- net LOAD_B2 renamed LOAD_B_C
- removed net LOAD_A1: J2.1, K12.S
- removed net LOAD_B1: J4.1, K22.S
- new net LOAD_A_NC: J2.1, K12.O
- new net LOAD_A_NO: J2.3, K12.S
- new net LOAD_B_NC: J4.1, K22.O
- new net LOAD_B_NO: J4.3, K22.S
